File: pcb/FireSide v2.5/FireSide v2.5.kicad_sch (KiCad schematic)
At the start: 34 parts, among them J1 Conn_01x02_Pin, J11 Conn_01x02_Pin, J12 Conn_01x02_Pin, J13 Screw_Terminal_01x03, J14 Screw_Terminal_01x02, J2 Conn_01x02_Pin, J3 Conn_01x02_Pin, J4 Conn_01x02_Pin, J5 Conn_01x02_Pin, J6 Conn_01x02_Pin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

Commit message: [FS] Updated PCB files to v2.5
Parts:
- added D1: YELLOW, LED_SMD:LED_0805_2012Metric, symbol Device:LED
- added D2: GREEN, LED_SMD:LED_0805_2012Metric, symbol Device:LED
- added J10: Conn_01x02_Pin, Connector_JST:JST_EH_B2B-EH-A_1x02_P2.50mm_Vertical, symbol Connector:Conn_01x02_Pin
- added J9: Screw_Terminal_01x03, TerminalBlock:TerminalBlock_bornier-3_P5.08mm, symbol Connector:Screw_Terminal_01x03
- added Q1: MMBT2222A, Package_TO_SOT_SMD:SOT-23, symbol Transistor_BJT:MMBT2222A
- added R1, R3: 165, Resistor_SMD:R_0805_2012Metric, symbol Device:R
- added R4: 1k, Resistor_SMD:R_0805_2012Metric, symbol Device:R
Connections:
- net 3.3V: now also J9.1 (Pin_1); no longer U2.1 (VDD)
- net GND: now also D1.1 (K), D2.1 (K), J9.2 (Pin_2), Q1.2 (E)
- net RX_RYLR: now also U9.CN3_1 (PA9/D1); no longer U9.CN3_2 (PA10/D0)
- net TX_RYLR: now also U9.CN3_2 (PA10/D0); no longer U9.CN3_1 (PA9/D1)
- net VI: now also J10.2 (Pin_2)
- net LAUNCH_LED: now reaches U9.CN3_5 (PA12/D2)
- net LAUNCH_LED: now also R3.2
- net ARM_LED: now reaches U9.CN3_7 (PB7/D4)
- net ARM_LED: now also R1.2
- net STATUS_PIN: now reaches U9.CN3_8 (PB6/D5)
- net STATUS_PIN: now also Q1.1 (B)
- new net: D1.2 (A), R1.1
- new net: Q1.3 (C), R4.1
- new net: J10.1 (Pin_1), R4.2
- new net: D2.2 (A), R3.1
- new net 3.3Vin: J9.3 (Pin_3), U2.1 (VDD)
- no-connect marks 21 -> 18
Other:
- note added: "3.3V"
- note added: "FSM LEDS"
- note added: "RYLR SWITCH"
- note added: "STATUS INDICATOR CIRCUIT"
- note removed: "3V"
- moved on the sheet: TP1, TP2
